File: PCB/hunter/hunter.kicad_pcb (KiCad board)
At the start: 2 copper layers, 36.2 x 52.6 mm, 1 part

Commit message: pcb first attempt
(cherry picked from commit e2accebbfe027ec41e787505fa792397e5ce38f1)
Parts:
- removed REF**: SW_SPST_PTS645, Button_Switch_SMD:SW_SPST_PTS645
- added AE1: Antenna, Connector_PinHeader_2.54mm:PinHeader_1x01_P2.54mm_Vertical, F.Cu at (52.9, 75.9)
- added C101: 27pF, Capacitor_SMD:C_0402_1005Metric, F.Cu at (84.8, 56.0)
- added C121: 6.8pF, Capacitor_SMD:C_0402_1005Metric, F.Cu at (52.0, 61.3)
- added C122: 12pF, Capacitor_SMD:C_0402_1005Metric, F.Cu at (51.7, 64.9)
- added C123: 6.8pF, Capacitor_SMD:C_0402_1005Metric, F.Cu at (51.9, 68.2)
- added C124: 220pF, Capacitor_SMD:C_0402_1005Metric, F.Cu at (51.1, 55.8)
- added C125: 220pF, Capacitor_SMD:C_0402_1005Metric, F.Cu at (52.5, 71.6)
- added C131: 6.8pF, Capacitor_SMD:C_0402_1005Metric, F.Cu at (55.1, 57.4)
- added C51: 100nF, Capacitor_SMD:C_0402_1005Metric, F.Cu at (57.2, 58.2)
- added C61: 10uF, Capacitor_Tantalum_SMD:CP_EIA-3216-18_Kemet-A, F.Cu at (82.9, 60.5)
- added C81: 27pF, Capacitor_SMD:C_0402_1005Metric, F.Cu at (75.7, 56.0)
- added D11: LED1, LED_SMD:LED_0603_1608Metric, F.Cu at (61.0, 73.6)
- added D2: LED2, LED_SMD:LED_0603_1608Metric, F.Cu at (75.7, 73.6)
- added J1: Battery, parts:MyBatteryConnector, F.Cu at (62.9, 98.0)
- added J2: JTAG, Connector_PinHeader_2.54mm:PinHeader_1x04_P2.54mm_Vertical, F.Cu at (79.6, 59.7)
- added L121: 33nH, Inductor_SMD:L_0402_1005Metric, F.Cu at (51.6, 57.6)
- added L122: 18nH, Inductor_SMD:L_0402_1005Metric, F.Cu at (53.4, 63.4)
- added L123: 33nH, Inductor_SMD:L_0402_1005Metric, F.Cu at (53.4, 66.5)
- added L131: 33nH, Inductor_SMD:L_0402_1005Metric, F.Cu at (54.5, 61.1)
- added R171: 56k, Resistor_SMD:R_0402_1005Metric, F.Cu at (54.8, 51.1)
- added SW1: SW_Light, Button_Switch_SMD:SW_SPST_Omron_B3FS-100xP, F.Cu at (68.1, 54.4)
- added SW2: SW_LightUp, Button_Switch_SMD:SW_SPST_Omron_B3FS-100xP, F.Cu at (61.0, 66.6)
- added SW3: SW_LightDown, Button_Switch_SMD:SW_SPST_Omron_B3FS-100xP, F.Cu at (75.6, 66.6)
- added SW4: SW_Fan, Button_Switch_SMD:SW_SPST_Omron_B3FS-100xP, F.Cu at (68.1, 80.4)
- added SW5: SW_FanUp, Button_Switch_SMD:SW_SPST_Omron_B3FS-100xP, F.Cu at (60.6, 92.7)
- added SW6: SW_FanDown, Button_Switch_SMD:SW_SPST_Omron_B3FS-100xP, F.Cu at (75.7, 92.7)
- added TP8: TestPoint, TestPoint:TestPoint_Pad_D1.0mm, F.Cu at (75.2, 52.2)
- added U1: CC1101RGPR, parts:CC1101RGPR, F.Cu at (58.7, 54.2)
- added U2: STM8L101F3U6TR, parts:STM8L101F3U6TR, F.Cu at (77.8, 80.0)
- added Y1: 26MHz, Crystal:Crystal_SMD_0603-4Pin_6.0x3.5mm, F.Cu at (80.4, 54.8)

Commit message: PCB wiring first attempt
Parts:
- removed TP8: TestPoint, TestPoint:TestPoint_Pad_D1.0mm
- Y1: footprint Crystal:Crystal_SMD_0603-4Pin_6.0x3.5mm -> Crystal:Crystal_SMD_3225-4Pin_3.2x2.5mm
- moved C81 22.4 mm to (54.9, 64.5), turned to 270 degrees
- moved C101 22.1 mm to (63.4, 61.9)
- moved Y1 21.1 mm to (60.2, 61.1)
- moved R171 4.19 mm to (58.9, 50.6), turned to 0 degrees
- moved J1 0.20 mm to (62.8, 97.9)
Connections:
- J1 pad +: (no net) -> +3V0
- J1 pad -: (no net) -> GND
- U1 pad V: (no net) -> GND
Routing:
- net +3V0: track 0.00 -> 93.4 mm, vias 0 -> 8
- net Net-(U1-Pad20): track 0.00 -> 58.2 mm, vias 0 -> 6
- net Net-(U1-Pad1): track 0.00 -> 54.9 mm, vias 0 -> 6
- net Net-(U1-Pad2): track 0.00 -> 45.1 mm, vias 0 -> 2
- net Net-(U1-Pad7): track 0.00 -> 38.9 mm, vias 0 -> 4
- net Net-(U1-Pad6): track 0.00 -> 38.3 mm, vias 0 -> 2
- net Net-(J2-Pad2): track 0.00 -> 32.5 mm
- net Net-(SW1-Pad1): track 0.00 -> 32.4 mm
- net Net-(J2-Pad4): track 0.00 -> 30.4 mm, vias 0 -> 2
- net Net-(SW2-Pad1): track 0.00 -> 27.6 mm, vias 0 -> 2
- net Net-(SW3-Pad1): track 0.00 -> 26.1 mm
- net Net-(SW5-Pad1): track 0.00 -> 25.7 mm
- net Net-(D2-Pad2): track 0.00 -> 25.5 mm, vias 0 -> 2
- net Net-(C131-Pad2): track 0.00 -> 22.5 mm, vias 0 -> 2
- net Net-(D11-Pad2): track 0.00 -> 21.1 mm, vias 0 -> 2
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